File: PCB/SatNOGS_Board/SatNOGSBoard.brd (EAGLE design)
At the start: 59.4 x 68.6 mm, 17 parts, among them J1 2, J2 3, J3 4

Commit message: Change the 1x8 header, change the names in tplace layer.
Parts:
- IO: device con-lsta:FE08 -> pinhead:1X08
- renumbered DRIVER1 to AZIMUTH, DRIVER2 to ELEVATION
Other:
- board text added: "AZIMUTH"
- board text added: "ELEVATION"
- board text removed: "Motor1"
- board text removed: "Motor2"
