File: PCB/satnogs_controller/satnogs_controller.sch (KiCad schematic (older format))
At the start: 13 parts, among them P1 CONN_01X04, P2 CONN_02X03, P3 CONN_02X02, P4 CONN_02X04, P5 CONN_01X18, SW1 RST, U1 Pro_Micro, U2 MAX485

Commit message: Update satnogs controller. Delete satnogs stepper driver. Add stepper driver in satnogs controller. Update 3d models and packages of satnogs library. Update BOM of satnogs controller.
Parts:
- added C3, C4: 100u, Capacitors_ThroughHole:C_Radial_D6.3_L11.2_P2.5, symbol CP
- added JP1, JP2, JP3, JP4, JP5, JP6: Jumper_NO_Small, Pin_Headers:Pin_Header_Straight_1x02, symbol Jumper_NO_Small
- added P6: CONN_01X02, Connect:bornier2, symbol CONN_01X02
- added P7, P8: CONN_01X04, Connect:bornier4, symbol CONN_01X04
- added R4, R7: 100k, Resistors_SMD:R_0805_HandSoldering, symbol R
- added R5, R6: 4.7k, Resistors_SMD:R_0805_HandSoldering, symbol R
- added U3, U4: POLOLU_A4988, satnogs:SWDIP8_.6W, symbol POLOLU_A4988
- C1: Distributor (none) -> Mouser 77-VJ0805Y104KXJCBC; Manufacturer (none) -> VJ0805Y104KXJCW1BC; Notes (none) -> 16VDC; Package (none) -> 0805; Price (none) -> 0.118€
- C2: Distributor (none) -> Mouser 667-ECA-1EM100B; Manufacturer (none) -> ECA-1EM100B; Notes (none) -> 10uF 25VDC 85C; Package (none) -> ThroughHole:C_Radial_D6.3_L11.2_P2.5; Price (none) -> 0.136€
- P1: Distributor (none) -> SparkFun PRT-00553; Manufacturer (none) -> -; Notes (none) -> https://www.sparkfun.com/products/553; Package (none) -> 1x40 pin right-angle PTH pitch 2.54; Price (none) -> 1.85€
- P2, P4: Distributor (none) -> SparkFun PRT-12791; Manufacturer (none) -> -; Notes (none) -> https://www.sparkfun.com/products/12791; Package (none) -> 2x23 pin male PTH header; Price (none) -> -
- P3: Distributor (none) -> SparkFun PRT-12791; Manufacturer (none) -> -; Notes (none) -> https://www.sparkfun.com/products/12791; Package (none) -> 2x23 pin male PTH header; Price (none) -> 0.9€
- P5, U1: Distributor (none) -> SparkFun PRT-00115; Manufacturer (none) -> -; Notes (none) -> https://www.sparkfun.com/products/115; Package (none) -> 1x40 female header PTH pitch 2.54; Price (none) -> 1.42€
- R1: Distributor (none) -> Mouser 71-CRCW0805120RJNEA; Manufacturer (none) -> CRCW0805120RJNEA; Notes (none) -> 1/8W 5%; Package (none) -> 0805; Price (none) -> 0.091€
- R2, R3: value R -> 4.7k; Distributor (none) -> Mouser 71-CRCW0805J-4.7K-E3; Manufacturer (none) -> CRCW08054K70JNEA; Notes (none) -> 1/8W 5%; Package (none) -> 0805; Price (none) -> 0.091€
- SW1: symbol SW_PUSH -> SW_PUSH-RESCUE-satnogs_controller; Distributor (none) -> SparkFun COM-08720; Manufacturer (none) -> -; Notes (none) -> https://www.sparkfun.com/products/8720; Package (none) -> -; Price (none) -> 0.9€
- U2: Distributor (none) -> Mouser 701-SP485CN-L; Manufacturer (none) -> SP485CN-L; Notes (none) -> Operating Supply Voltage: 5 V; Package (none) -> SOIC-8 Narrow; Price (none) -> 0.86€
Connections:
- net labels added: 1AM1, 1AM2, 1BM1, 1BM2, 2AM1, 2AM2, 2BM1, 2BM2, D15, DC_MOTORS, I2C-1, I2C-2/DevPins, M1IN1->DIRM1->D6, M1IN2->STEPM1->D5, M2IN1->DIRM2->D10, M2IN2->STEPM2->D9, MS1M1, MS1M2, Note, POWER_IN, RST, SCL1, SCL2, SDA1, SDA2, STEPPER_MOTOR1, STEPPER_MOTOR2, VMOT
- net labels removed: CLK, CS, DO, Encoder/SPI/DevPins, I2C, MotorHeader, SCL, SDA
- wire segments 109 -> 166
- no-connect marks 3 -> 1
Other:
- moved on the sheet: C1, C2, P1, P2, P4, U2

Commit message: Update satnogs controller. Replace arduino micro with arduino pro mini. Fix wrong connection with RX-TX in SP485CN (RS485). Better pin-header arrangement.
Parts:
- removed P3: CONN_02X02, Pin_Headers:Pin_Header_Straight_2x02, symbol CONN_02X02
- removed SW1: RST, satnogs:smd_push2, symbol SW_PUSH-RESCUE-satnogs_controller
- removed U1: Pro_Micro, satnogs:Pro_Micro, symbol Pro_Micro
- added D1: ZENERsmall, Diodes_ThroughHole:Diode_DO-41_SOD81_Horizontal_RM10, symbol ZENERsmall
- added P9: CONN_02X02, Pin_Headers:Pin_Header_Straight_2x02, symbol CONN_02X02
- added R8, R9: 4.7k, Resistors_SMD:R_0805_HandSoldering, symbol R
- added U1: Pro_Mini, satnogs:pro-mini, symbol Pro_Mini
Connections:
- net labels added: A2, A3
- net labels removed: D15, DC_MOTORS, EndStops, I2C-1, I2C-2/DevPins, M1IN1->DIRM1->D6, M1IN2->STEPM1->D5, M2IN1->DIRM2->D10, M2IN2->STEPM2->D9, Microcontroller, Note, POWER_IN, RS485, RST, STEPPER_MOTOR1, STEPPER_MOTOR2
- wire segments 166 -> 153
- no-connect marks 1 -> 6
Other:
- note added: "DC Motors"
- note added: "Dev pins"
- note added: "EndStops"
- note added: "I2C-1,2"
- note added: "M1IN1->DIRM1->D6\nM1IN2->STEPM1->D5\nM2IN1->DIRM2-D10\nM2IN2->STEPM2->D9"
- note added: "Microcontroller"
- note added: "Power In for stepper motors"
- note added: "RS485"
- note added: "Regulator in pro-mini, is MIC5205:\n5V@150mA\nReverse-current protection"
- note added: "Stepper motor 1"
- note added: "Stepper motor 2"
- moved on the sheet: C1, C2, C3, C4, JP1, JP2, JP3, JP4, JP5, JP6, P1, P2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

Commit message: Update BOM's.
Parts:
- D1: Distributor (none) -> Mouser 512-BZX85C10; Manufacturer (none) -> BZX85C10; Notes (none) -> 10V-1W; Package (none) -> DO-41; Price (none) -> 0.192€
- P1: value CONN_01X04 -> RS485
- P2: value CONN_02X03 -> End-Stops
- P4: value CONN_02X04 -> I2C
- P5: value CONN_01X18 -> DC Motors Driver
- P6: value CONN_01X02 -> Power-IN
- P7: value CONN_01X04 -> Motor1
- P8: value CONN_01X04 -> Motor2
- P9: value CONN_02X02 -> Dev-Pins; Distributor (none) -> SparkFun PRT-12791; Manufacturer (none) -> -; Notes (none) -> https://www.sparkfun.com/products/12791; Package (none) -> -; Price (none) -> -
- U1: Distributor (none) -> SparkFun PRT-00115; Manufacturer (none) -> -; Notes (none) -> https://www.sparkfun.com/products/115; Package (none) -> 1x40 female header PTH pitch 2.54; Price (none) -> 1.42€
Other:
- note added: "Failsafe-biasing network for \nlegacy transceivers like SP485CN-L\n"
- note added: "Regulator in pro-mini, is MIC5205:\n5V@150mA with reverse-current protection"
- note removed: "Regulator in pro-mini, is MIC5205:\n5V@150mA\nReverse-current protection"
Changed lines of the file:
@@
 P 10030 3155
 F 0 "P5" H 10030 4105 50  0000 C CNN
-F 1 "CONN_01X18" V 10130 3155 50  0000 C CNN
+F 1 "DC Motors Driver" V 10130 3155 50  0000 C CNN
 F 2 "satnogs:pin_socket_18" H 10030 3155 60  0001 C CNN
 F 3 "-" H 10030 3155 60  0001 C CNN
@@
 P 1615 1850
 F 0 "P1" H 1615 2100 50  0000 C CNN
-F 1 "CONN_01X04" V 1715 1850 50  0000 C CNN
+F 1 "RS485" V 1715 1850 50  0000 C CNN
 F 2 "Pin_Headers:Pin_Header_Angled_1x04" H 1615 1850 60  0001 C CNN
 F 3 "-" H 1615 1850 60  0001 C CNN
@@
 P 8000 1685
 F 0 "P4" H 8000 1935 50  0000 C CNN
-F 1 "CONN_02X04" H 8000 1435 50  0000 C CNN
+F 1 "I2C" H 8000 1435 50  0000 C CNN
 F 2 "Pin_Headers:Pin_Header_Straight_2x04" H 8000 485 60  0001 C CNN
 F 3 "https://cdn.sparkfun.com/datasheets/Prototyping/16188.pdf" H 8000 485 60  0001 C CNN
@@
 P 6200 1675
 F 0 "P2" H 6200 1875 50  0000 C CNN
-F 1 "CONN_02X03" H 6200 1475 50  0000 C CNN
+F 1 "End-Stops" H 6200 1475 50  0000 C CNN
 F 2 "Pin_Headers:Pin_Header_Straight_2x03" H 6200 475 60  0001 C CNN
 F 3 "https://cdn.sparkfun.com/datasheets/Prototyping/16188.pdf" H 6200 475 60  0001 C CNN
@@
 P 3185 5000
 F 0 "P7" H 3185 5250 50  0000 C CNN
-F 1 "CONN_01X04" V 3285 5000 50  0000 C CNN
+F 1 "Motor1" V 3285 5000 50  0000 C CNN
 F 2 "Connect:bornier4" H 3185 5000 50  0001 C CNN
 F 3 "https://www.sparkfun.com/datasheets/Prototyping/Screw-Terminal-5mm.pdf" H 3185 5000 50  0001 C CNN
@@
 P 7095 5000
 F 0 "P8" H 7095 5250 50  0000 C CNN
-F 1 "CONN_01X04" V 7195 5000 50  0000 C CNN
+F 1 "Motor2" V 7195 5000 50  0000 C CNN
 F 2 "Connect:bornier4" H 7095 5000 50  0001 C CNN
 F 3 "https://www.sparkfun.com/datasheets/Prototyping/Screw-Terminal-5mm.pdf" H 7095 5000 50  0001 C CNN
@@
 P 1545 5030
 F 0 "P6" H 1545 5180 50  0000 C CNN
-F 1 "CONN_01X02" V 1645 5030 50  0000 C CNN
+F 1 "Power-IN" V 1645 5030 50  0000 C CNN
 F 2 "Connect:bornier2" H 1545 5030 50  0001 C CNN
 F 3 "https://www.sparkfun.com/datasheets/Prototyping/Screw-Terminal-5mm.pdf" H 1545 5030 50  0001 C CNN
@@
 F 1 "Pro_Mini" H 5670 2255 60  0000 C CNN
 F 2 "satnogs:pro-mini" H 5660 3095 60  0001 C CNN
-F 3 "" H 5660 3095 60  0000 C CNN
+F 3 "-" H 5660 3095 60  0001 C CNN
+F 4 "SparkFun PRT-00115" H 5660 3195 60  0001 C CNN "Distributor"
+F 5 "-" H 5660 3195 60  0001 C CNN "Manufacturer"
+F 6 "1x40 female header PTH pitch 2.54" H 5660 3195 60  0001 C CNN "Package"
+F 7 "https://www.sparkfun.com/products/115" H 5660 3195 60  0001 C CNN "Notes"
+F 8 "1.42€" H 5660 3195 60  0001 C CNN "Price"
 	1    5660 3195
 	1    0    0    -1
@@
 F 1 "ZENERsmall" H 2325 1750 50  0000 C CNN
 F 2 "Diodes_ThroughHole:Diode_DO-41_SOD81_Horizontal_RM10" H 2325 1850 50  0001 C CNN
-F 3 "" H 2325 1850 50  0000 C CNN
+F 3 "http://www.mouser.com/ds/2/149/BZX85C10-888846.pdf" H 2325 1850 50  0001 C CNN
+F 4 "Mouser 512-BZX85C10" H 2325 1850 60  0001 C CNN "Distributor"
+F 5 "BZX85C10" H 2325 1850 60  0001 C CNN "Manufacturer"
+F 6 "DO-41" H 2325 1850 60  0001 C CNN "Package"
+F 7 "10V-1W" H 2325 1850 60  0001 C CNN "Notes"
+F 8 "0.192€" H 2325 1850 60  0001 C CNN "Price"
 	1    2325 1850
 	0    1    1    0
@@
 A2
 Text Notes 6810 2580 0    61   ~ 0
-Regulator in pro-mini, is MIC5205:\n5V@150mA\nReverse-current protection
+Regulator in pro-mini, is MIC5205:\n5V@150mA with reverse-current protection
 $Comp
 L CONN_02X02 P9
@@
 P 4370 1585
 F 0 "P9" H 4370 1735 50  0000 C CNN
-F 1 "CONN_02X02" H 4370 1435 50  0000 C CNN
+F 1 "Dev-Pins" H 4370 1435 50  0000 C CNN
 F 2 "Pin_Headers:Pin_Header_Straight_2x02" H 4370 385 50  0001 C CNN
-F 3 "" H 4370 385 50  0000 C CNN
+F 3 "https://cdn.sparkfun.com/datasheets/Prototyping/16188.pdf" H 4370 385 50  0001 C CNN
+F 4 "SparkFun PRT-12791" H 4370 1585 60  0001 C CNN "Distributor"
+F 5 "-" H 4370 1585 60  0001 C CNN "Manufacturer"
+F 6 "-" H 4370 1585 60  0001 C CNN "Package"
+F 7 "https://www.sparkfun.com/products/12791" H 4370 1585 60  0001 C CNN "Notes"
+F 8 "-" H 4370 1585 60  0001 C CNN "Price"
 	1    4370 1585
 	1    0    0    -1
@@
 NoConn ~ 6290 3545
 NoConn ~ 6290 3645
+Text Notes 1450 4140 0    61   ~ 0
+Failsafe-biasing network for \nlegacy transceivers like SP485CN-L\n
 $EndSCHEMATC

Commit message: Updates in rotator controller.
Add RJ45 for communication and power in (PoE).
New dimensions of board (euroboard 100x80 mm)
Embed the power supply to the board (WIP).
Add pins for indicator LED and for rf switch (optional).
Add additional pads for power in case that PoE (RJ45) isn't suitable.
Updates in schematic and board wuth new library parts.
Parts:
- removed C2: 10u, Capacitors_ThroughHole:C_Radial_D6.3_L11.2_P2.5, symbol CP
- removed D1: ZENERsmall, Diodes_ThroughHole:Diode_DO-41_SOD81_Horizontal_RM10, symbol ZENERsmall
- removed P1: RS485, Pin_Headers:Pin_Header_Angled_1x04, symbol CONN_01X04
- removed P5: DC Motors Driver, satnogs:pin_socket_18, symbol CONN_01X18
- removed P6: Power-IN, Connect:bornier2, symbol CONN_01X02
- removed P9: Dev-Pins, Pin_Headers:Pin_Header_Straight_2x02, symbol CONN_02X02
- removed U1: Pro_Mini, satnogs:pro-mini, symbol Pro_Mini
- added C2: 2.2u, Capacitors_SMD:C_1210, symbol C_Small
- added C5: 10u, Capacitors_ThroughHole:C_Radial_D6.3_L11.2_P2.5, symbol CP
- added C6: 100n, Capacitors_SMD:C_0805_HandSoldering, symbol C_Small
- added C7: 7.5n, Capacitors_SMD:C_0805_HandSoldering, symbol C_Small
- added C8: 10p, Capacitors_SMD:C_0805_HandSoldering, symbol C_Small
- added C9: 47u, Capacitors_SMD:C_1210, symbol C_Small
- added D1, D2: D_Schottky, Diodes_SMD:DO-214AB, symbol D_Schottky
- added F1: FUSE, SMD_Packages:Fuse_SMD, symbol FUSE
- added FB1: FILTER, Resistors_SMD:R_0805_HandSoldering, symbol FILTER
- added J1: RJ45, Connect:RJ45_8, symbol RJ45
- added JP7, JP8, JP9: Jumper_NO_Small, Resistors_SMD:R_0805_HandSoldering, symbol Jumper_NO_Small
- added L1: 27u, satnogs:bourns-srr1210, symbol INDUCTOR_SMALL
- added P1: Dev-Pins, Pin_Headers:Pin_Header_Straight_2x03, symbol CONN_02X03
- added P3: Power-In, Wire_Connections_Bridges:WireConnection_2.00mmDrill, symbol CONN_01X02
- added R10: 221k, Resistors_SMD:R_0805_HandSoldering, symbol R
- added R11: 26.7k, Resistors_SMD:R_0805_HandSoldering, symbol R
- added R12: 147k, Resistors_SMD:R_0805_HandSoldering, symbol R
- added R13: 10.5k, Resistors_SMD:R_0805_HandSoldering, symbol R
- added U1: ARDUINO_PRO_MINI, satnogs:arduino-pro-mini, symbol ARDUINO_PRO_MINI
- added U5: TPS54360DDA, satnogs:HSOP-8, symbol TPS54360DDA
- added U6: POLOLU_DUAL_MC33926, satnogs:pololu-dual-mc33926, symbol POLOLU_DUAL_MC33926
- JP1, JP2, JP3, JP4, JP5, JP6: footprint Pin_Headers:Pin_Header_Straight_1x02 -> Resistors_SMD:R_0805_HandSoldering
- U3, U4: footprint satnogs:SWDIP8_.6W -> satnogs:pololu-a4988
Connections:
- net labels added: +12V, FB, M1D1, M1D2, M1RST, M1SLP, M2D1, M2D2, M2RST, M2SLP, MS2M1, MS2M2, MS3M1, MS3M2, PB5, VIN_RJ45
- net labels removed: VMOT
- wire segments 153 -> 207
- no-connect marks 6 -> 13
Other:
- note added: "802.3af Standards\nT568A color\n10/100 mode B, DC on spares"
- note added: "Input Connector"
- note added: "Input from PoE 24W, 24V@1A"
- note added: "M1IN1->STEPM1->D6\nM1IN2->DIRM1->D5\nM2IN1->STEPM2->D10\nM2IN2->DIRM2->D9"
- note added: "Note for microstepping\nMS1 MS2 MS3 Microstep Resolution\nLow Low Low Full step\nHigh Low Low Half step\nLow High Low Quarter step\nHigh High Low Eighth step\nHigh High High Sixteenth step"
- note added: "Output: 12V@3.5A"
- note added: "Power Supply Module"
- note added: "SLEW/INV default state: GND"
- note added: "Separate chasis connector for power-in.\nIn case that the PoE isn't suitable."
- note added: "Solder to have UART\nas communication"
- note removed: "M1IN1->DIRM1->D6\nM1IN2->STEPM1->D5\nM2IN1->DIRM2-D10\nM2IN2->STEPM2->D9"
- note removed: "Power In for stepper motors"
- moved on the sheet: C1, C3, C4, JP1, JP2, JP3, JP4, JP5, JP6, P2, P4, P7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

Commit message: Updates in PCB and schematic.
Add digital and power ground planes (WIP).
Connection of separate GND with zero resistor.
Add I2C multiplexer.
Finalize power supply of 12V.
Change RJ45 to headers.
Add RC filter (LPF) for end-stops.
Add more dev-pins.
Add filter in uC voltage input.

Signed-off-by: zisi <agzisim@gmail.com>
Parts:
- removed J1: RJ45, Connect:RJ45_8, symbol RJ45
- removed JP9: Jumper_NO_Small, Resistors_SMD:R_0805_HandSoldering, symbol Jumper_NO_Small
- removed P1: Dev-Pins, Pin_Headers:Pin_Header_Straight_2x03, symbol CONN_02X03
- removed P3: Power-In, Wire_Connections_Bridges:WireConnection_2.00mmDrill, symbol CONN_01X02
- added C10, C11, C12: 0.1u, Capacitors_SMD:C_0805_HandSoldering, symbol C_Small
- added FB2: FILTER, Resistors_SMD:R_0805_HandSoldering, symbol FILTER
- added JP10: Jumper_NO_Small, Resistors_SMD:R_0805_HandSoldering, symbol Jumper_NO_Small
- added P1: DEV-PINS, Pin_Headers:Pin_Header_Straight_2x04, symbol CONN_02X04
- added P3: RJ45, Pin_Headers:Pin_Header_Straight_2x04, symbol CONN_02X04
- added R14, R15: 200, Resistors_SMD:R_0805_HandSoldering, symbol R
- added R16, R17: 4.7k, Resistors_SMD:R_0805_HandSoldering, symbol R
- added U7: PCA9540B, Housings_SSOP:TSSOP-8_3x3mm_Pitch0.65mm, symbol PCA9540B
- C1: Distributor Mouser 77-VJ0805Y104KXJCBC -> (none); Manufacturer VJ0805Y104KXJCW1BC -> (none); Mnf. (none) -> VJ0805Y104KXJCW1BC; Notes 16VDC -> (none); Package 0805 -> (none); Price 0.118€ -> 0.118
- C2: Mnf. (none) -> C3225X7R2A225K230AB; Price (none) -> 0.697
- C3, C4: footprint Capacitors_ThroughHole:C_Radial_D6.3_L11.2_P2.5 -> Capacitors_SMD:c_elec_6.3x5.3; Distributor Mouser 667-ECA-1VM101 -> (none); Manufacturer ECA-1VM101 -> (none); Mnf. (none) -> EXV107M016A9GAA; Notes 100u 35V 85C -> (none); Package ThroughHole:C_Radial_D6.3_L11.2_P2.5 -> (none); Price 0.235€ -> 0.443
- C5: footprint Capacitors_ThroughHole:C_Radial_D6.3_L11.2_P2.5 -> Capacitors_SMD:c_elec_6.3x5.3; Distributor Mouser 667-ECA-1EM100B -> (none); Manufacturer ECA-1EM100B -> (none); Mnf. (none) -> EXV107M016A9GAA; Notes 10uF 25VDC 85C -> (none); Package ThroughHole:C_Radial_D6.3_L11.2_P2.5 -> (none); Price 0.136€ -> 0.443
- C6: Mnf. (none) -> 08053C104KAT2A; Price (none) -> 0.091
- C7: Mnf. (none) -> GRM2195C1H752JA01D; Price (none) -> 0.244
- C8: Mnf. (none) -> C0805C100K5GACTU; Price (none) -> 0.091
- C9: Mnf. (none) -> GRM32ER61C476ME15L; Price (none) -> 0.851
- D1, D2: Mnf. (none) -> B560C-13-F; Price (none) -> 0.494
- F1: footprint SMD_Packages:Fuse_SMD -> satnogs:mini-fuse-holder-3568; Mnf. (none) -> Keystone Electronics, 3568; Price (none) -> 0.732
- FB1: Mnf. (none) -> MPZ2012S300A; Price (none) -> 0.109
- JP1, JP2, JP3, JP4, JP5, JP6, JP7, JP8: Distributor SparkFun PRT-12791 -> (none); Manufacturer - -> (none); Notes https://www.sparkfun.com/products/12791 -> (none); Package 2x23 pin male PTH header -> (none); Price - -> (none)
- L1: Mnf. (none) -> SRR1210-270M; Price (none) -> 1
- P7, P8: Distributor SparkFun PRT-08432 -> (none); Manufacturer - -> (none); Mnf. (none) -> Altech - 30.704; Notes https://www.sparkfun.com/products/8432 -> (none); Package 5mm Pitch 4-Pin -> (none); Price 1.8€ -> 1.99
- R1: Distributor Mouser 71-CRCW0805120RJNEA -> (none); Manufacturer CRCW0805120RJNEA -> (none); Mnf. (none) -> CRCW0805120RJNEA; Notes 1/8W 5% -> (none); Package 0805 -> (none); Price 0.091€ -> 0.091
- R10: Mnf. (none) -> CRCW0805221KFKEA; Price (none) -> 0.091
- R11: Mnf. (none) -> CRCW080526K7FKEA; Price (none) -> 0.091
- R12: Mnf. (none) -> CRCW0805147KFKEA; Price (none) -> 0.091
- R13: Mnf. (none) -> CRCW080510K5FKEA; Price (none) -> 0.091
- R2, R3, R5, R6, R8: Distributor Mouser 71-CRCW0805J-4.7K-E3 -> (none); Manufacturer CRCW08054K70JNEA -> (none); Mnf. (none) -> CRCW08054K70JNEA; Notes 1/8W 5% -> (none); Package 0805 -> (none); Price 0.091€ -> 0.091
- R4: Distributor Mouser 71-CRCW0805J-100K-E3 -> (none); Manufacturer CRCW0805100KJNEA -> (none); Mnf. (none) -> CRCW0805100KJNEA; Package 0805 -> (none); Price 0.091€ -> 0.091
- R7: Distributor Mouser 71-CRCW0805J-100K-E3 -> (none); Manufacturer CRCW0805100KJNEA -> (none); Mnf. (none) -> CRCW0805100KJNEA; Notes 1/8W 5% -> (none); Package 0805 -> (none); Price 0.091€ -> 0.091
- R9: Distributor Mouser 71-CRCW0805J-4.7K-E3 -> (none); Notes 1/8W 5% -> (none); Package 0805 -> (none); Price 0.091€ -> 0.091
- U1: Mnf. (none) -> Sparkfun - DEV-11113; Price (none) -> 9.5
- U2: Distributor Mouser 701-SP485CN-L -> (none); Notes Operating Supply Voltage: 5 V -> (none); Package SOIC-8 Narrow -> (none); Price 0.86€ -> 0.86
- U3: Distributor SparkFun PRT-00115 -> (none); Manufacturer - -> (none); Mnf. (none) -> 1182; Notes https://www.sparkfun.com/products/115 -> (none); Package 1x40 female header PTH pitch 2.54 -> (none); Price 1.42€ -> 5.95
- U4: Distributor SparkFun PRT-00115 -> (none); Manufacturer - -> (none); Mnf. (none) -> 1182; Notes https://www.sparkfun.com/products/115 -> (none); Package 1x40 female header PTH pitch 2.54 -> (none); Price - -> 5.95
- U5: Mnf. (none) -> TPS54360DDAR; Price (none) -> 4.53
- U6: Mnf. (none) -> 1213; Price (none) -> 27.83
Connections:
- net labels added: BOOT, COMP, GNDD, PB3, PB4, RST, RT/CLK, SCL, SCL0, SDA, SDA0, SW, SW1_F, SW2_F, SW_VIN
- net labels removed: SCL2, SDA2, VIN_RJ45
- wire segments 207 -> 231
- no-connect marks 13 -> 10
Other:
- note added: "Debouncing filter\nfor the mechanichal\nend-stops.\n"
- note added: "Filter switching regulator\nfor 5V LDO"
- note added: "I2C-Multiplexer"
- note added: "VIN: 12 - 60V"
- note removed: "I2C-1,2"
- note removed: "Separate chasis connector for power-in.\nIn case that the PoE isn't suitable."
- moved on the sheet: C1, C2, C3, C4, C5, C6, C7, C8, C9, D1, D2, F1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
